File: schematics/GameOfLife/GameOfLife.sch (KiCad schematic (older format))
At the start: 139 parts, among them U1 74HC595, U2 CD74HC4067M

Commit message: Update schematics
Signed-off-by: Manuel Genovés <manuel.genoves@gmail.com>
Parts:
- gave numbers to parts that had none: 1
Connections:
- net at R10.1, R11.1, R12.1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: no longer D16.2 (A), R24.2
- new net: D16.2 (A), R24.2
Changed lines of the file:
@@
 Wire Wire Line
 	3300 4450 3300 5050
-Wire Wire Line
-	2300 6850 2500 6850
-Connection ~ 2300 6850
-Connection ~ 2500 6850
 Connection ~ 2800 2650
 Wire Wire Line
@@
 	5800 6250 5800 6850
 $Comp
-L MCU_Module:Arduino_Nano_v3.x A?
+L MCU_Module:Arduino_Nano_v3.x A1
 U 1 1 5F6A3660
 P 8850 2950
-F 0 "A?" H 8850 1861 50  0000 C CNN
+F 0 "A1" H 8850 1861 50  0000 C CNN
 F 1 "Arduino_Nano_v3.x" H 8850 1770 50  0000 C CNN
 F 2 "Module:Arduino_Nano" H 8850 2950 50  0001 C CIN
