File: schematics/GameOfLife/GameOfLife.kicad_pcb (KiCad board)
At the start: 2 copper layers, 139 parts, among them U1 74HC595, U2 CD74HC4067M

Commit message: Update schematics
Signed-off-by: Manuel Genovés <manuel.genoves@gmail.com>
Parts:
- moved U2 132.4 mm to (170.2, 207.0), turned to 180 degrees
- moved A1 79.0 mm to (96.5, 222.2), turned to 90 degrees
- moved U1 51.6 mm to (158.8, 201.9)
Connections:
- R10 pad 1: Net-(D16-Pad2) -> Net-(R10-Pad1)
- R11 pad 1: Net-(D16-Pad2) -> Net-(R10-Pad1)
- R12 pad 1: Net-(D16-Pad2) -> Net-(R10-Pad1)
- R13 pad 1: Net-(D16-Pad2) -> Net-(R10-Pad1)
- R14 pad 1: Net-(D16-Pad2) -> Net-(R10-Pad1)
- R15 pad 1: Net-(D16-Pad2) -> Net-(R10-Pad1)
- R16 pad 1: Net-(D16-Pad2) -> Net-(R10-Pad1)
- R9 pad 1: Net-(D16-Pad2) -> Net-(R10-Pad1)
- U1 pad 7: Net-(D16-Pad2) -> Net-(R10-Pad1)
Routing:
- net Net-(D1-Pad1): track 0.00 -> 141.5 mm
- net Net-(D10-Pad1): track 0.00 -> 119.9 mm
- net Net-(D11-Pad1): track 0.00 -> 100.9 mm
- net Net-(D12-Pad1): track 0.00 -> 81.8 mm
- net Net-(D16-Pad1): track 0.00 -> 79.6 mm
- net Net-(D15-Pad1): track 0.00 -> 69.9 mm
- net Net-(D13-Pad1): track 0.00 -> 62.8 mm
- net Net-(R10-Pad1): track 0.00 -> 61.5 mm
- net Net-(R17-Pad1): track 0.00 -> 50.1 mm
- net Net-(R65-Pad1): track 0.00 -> 49.3 mm
- net Net-(D14-Pad1): track 0.00 -> 43.7 mm
- net Net-(R57-Pad1): track 0.00 -> 34.8 mm
- net Net-(R25-Pad1): track 0.00 -> 24.7 mm
- net Net-(R33-Pad1): track 0.00 -> 21.9 mm
- net Net-(R49-Pad1): track 0.00 -> 19.6 mm
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
Commit message: Update pcb
Parts:
- removed U2: CD74HC4067M, Package_SO:SOIC-24W_7.5x15.4mm_P1.27mm
- added TB1: BOB-09056, GameOfLife:XDCR_BOB-09056, F.Cu at (175.3, 214.6)
- moved A1 40.4 mm to (68.6, 193.0), turned to 0 degrees
- moved U1 8.13 mm to (152.4, 207.0)
Connections:
- A1 pad 1: (no net) -> Net-(A1-Pad1)
- A1 pad 10: (no net) -> Net-(A1-Pad10)
- A1 pad 12: (no net) -> Net-(A1-Pad12)
- A1 pad 13: (no net) -> Net-(A1-Pad13)
- A1 pad 16: (no net) -> Net-(A1-Pad16)
- A1 pad 17: (no net) -> Net-(A1-Pad17)
- A1 pad 18: (no net) -> Net-(A1-Pad18)
- A1 pad 2: (no net) -> Net-(A1-Pad2)
- A1 pad 20: (no net) -> Net-(A1-Pad20)
- A1 pad 21: (no net) -> Net-(A1-Pad21)
- A1 pad 22: (no net) -> Net-(A1-Pad22)
- A1 pad 23: (no net) -> Net-(A1-Pad23)
- A1 pad 24: (no net) -> Net-(A1-Pad24)
- A1 pad 25: (no net) -> Net-(A1-Pad25)
- A1 pad 26: (no net) -> Net-(A1-Pad26)
- A1 pad 28: (no net) -> Net-(A1-Pad28)
- A1 pad 3: (no net) -> Net-(A1-Pad3)
- A1 pad 30: (no net) -> Net-(A1-Pad30)
- A1 pad 4: (no net) -> Net-(A1-Pad4)
- A1 pad 8: (no net) -> Net-(A1-Pad8)
- A1 pad 9: (no net) -> Net-(A1-Pad9)
- U1 pad 9: (no net) -> Net-(U1-Pad9)
Routing:
- net Net-(A1-Pad29): track 0.00 -> 137.4 mm
- net Net-(A1-Pad27): track 0.00 -> 114.0 mm
- net Net-(A1-Pad5): track 0.00 -> 112.7 mm
- net Net-(A1-Pad6): track 0.00 -> 109.5 mm
- net Net-(A1-Pad7): track 0.00 -> 105.5 mm
- net Net-(A1-Pad14): track 0.00 -> 102.7 mm
- net Net-(A1-Pad19): track 0.00 -> 89.1 mm
- net Net-(A1-Pad15): track 0.00 -> 81.4 mm
- net Net-(A1-Pad11): track 0.00 -> 79.9 mm
- net Net-(D14-Pad1): track 43.7 -> 103.2 mm
- net Net-(D13-Pad1): track 62.8 -> 121.0 mm
- net Net-(D12-Pad1): track 81.8 -> 138.7 mm
- net Net-(D11-Pad1): track 100.9 -> 156.5 mm
- net Net-(D10-Pad1): track 119.9 -> 174.3 mm
- net Net-(D1-Pad1): track 141.5 -> 192.8 mm
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