File: schematics/GameOfLife/_autosave-GameOfLife.sch (KiCad schematic (older format))
At the start: 139 parts, among them U1 74HC595

Commit message: Update pcb
Parts:
- gave numbers to parts that had none: 1
Changed lines of the file:
@@
 $EndComp
 $Comp
-L BOB-09056:BOB-09056 TB?
+L BOB-09056:BOB-09056 TB1
 U 1 1 5EF45707
 P 7250 3550
-F 0 "TB?" H 7250 5317 50  0000 C CNN
+F 0 "TB1" H 7250 5317 50  0000 C CNN
 F 1 "BOB-09056" H 7250 5226 50  0000 C CNN
 F 2 "XDCR_BOB-09056" H 7250 3550 50  0001 L BNN
